Commit message: fix: hardware interface error

File: p3dx_description/urdf/pioneer3dx_wheel.xacro (robot description, xacro)
@@ -16,6 +16,5 @@
 work original in ucs-ros-pkg.
  -->
-<robot
-	xmlns:xacro="http://ros.org/wiki/xacro">
+<robot xmlns:xacro="http://ros.org/wiki/xacro">
 	<!-- properties (constants) -->
 	<xacro:property name="M_PI" value="3.14159" />
@@ -82,5 +81,7 @@
 		<transmission name="${parent}_${suffix}_wheel_trans">
 			<type>pr2_mechanism_model/SimpleTransmission</type>
-			<joint name="base_${suffix}_wheel_joint" />
+			<joint name="base_${suffix}_wheel_joint">
+				<hardwareInterface>hardware_interface/EffortJointInterface</hardwareInterface>
+			</joint>
 			<actuator name="base_${suffix}_wheel_motor">
 				<hardwareInterface>EffortJointInterface</hardwareInterface>
